Commit message: add table model and update urdf

File: turtlebot3_description/urdf/turtlebot3_burger.gazebo.xacro (robot description, xacro)
@@ -4,4 +4,7 @@
   <xacro:arg name="imu_visual"   default="false"/>
   <gazebo reference="base_link">
+    <material>Gazebo/DarkGrey</material>
+  </gazebo>
+  <gazebo reference="table_link">
     <material>Gazebo/DarkGrey</material>
   </gazebo>

File: turtlebot3_description/urdf/turtlebot3_burger.urdf.xacro (robot description, xacro)
@@ -30,4 +30,31 @@
                izz="2.0064271e-03" />
     </inertial>
+  </link>
+  <joint name="table_joint" type="fixed">
+    <parent link="base_link"/>
+    <child link="table_link"/>
+    <origin xyz="-0.032 0.0 0.194" rpy="0 0 0"/>
+  </joint>
+  <link name="table_link">
+    <visual>
+      <origin xyz="0 0 0" rpy="0 0 0"/>
+      <geometry>
+        <mesh filename="package://turtlebot3_description/meshes/table/burger_table.stl" scale="0.001 0.001 0.001"/>
+      </geometry>
+      <material name="light_black"/>
+    </visual>
+    <collision>
+      <origin xyz="0 0 0" rpy="0 0 0"/>
+      <geometry>
+        <box size="0.140 0.140 0.009 "/>
+      </geometry>
+    </collision>
+    <inertial>
+      <origin xyz="0 0 0" rpy="0 0 0"/>
+      <mass value="0.0995"/>
+      <inertia ixx="1.92366666667e-04" ixy="0" ixz="0"
+               iyy="1.92366666667e-04" iyz="0"
+               izz="3.25033333333e-04" />
+      </inertial>
   </link>
   <joint name="wheel_left_joint" type="continuous">

Commit message: add camera and scan fileter

File: turtlebot3_description/urdf/turtlebot3_burger.gazebo.xacro (robot description, xacro)
@@ -2,4 +2,5 @@
 <robot name="turtlebot3_burger_sim" xmlns:xacro="http://ros.org/wiki/xacro">
   <xacro:arg name="laser_visual" default="false"/>
+  <xacro:arg name="camera_visual" default="false"/>
   <xacro:arg name="imu_visual"   default="false"/>
   <gazebo reference="base_link">
@@ -127,3 +128,36 @@
     </sensor>
   </gazebo>
+  <!--link : https://www.raspberrypi.org/documentation/hardware/camera/-->
+  <gazebo reference="camera_rgb_frame">
+    <sensor type="camera" name="Pi Camera">
+      <always_on>true</always_on>
+      <visualize>$(arg camera_visual)</visualize>
+      <camera>
+          <horizontal_fov>1.085595</horizontal_fov>
+          <image>
+              <width>320</width>
+              <height>240</height>
+              <format>R8G8B8</format>
+          </image>
+          <clip>
+              <near>0.03</near>
+              <far>100</far>
+          </clip>
+      </camera>
+      <plugin name="camera_controller" filename="libgazebo_ros_camera.so">
+        <alwaysOn>true</alwaysOn>
+        <updateRate>30.0</updateRate>
+        <cameraName>camera</cameraName>
+        <frameName>camera_rgb_optical_frame</frameName>
+        <imageTopicName>image</imageTopicName>
+        <cameraInfoTopicName>camera_info</cameraInfoTopicName>
+        <hackBaseline>0.07</hackBaseline>
+        <distortionK1>0.0</distortionK1>
+        <distortionK2>0.0</distortionK2>
+        <distortionK3>0.0</distortionK3>
+        <distortionT1>0.0</distortionT1>
+        <distortionT2>0.0</distortionT2>
+      </plugin>
+    </sensor>
+  </gazebo>
 </robot>

File: turtlebot3_description/urdf/turtlebot3_burger.urdf.xacro (robot description, xacro)
@@ -167,3 +167,28 @@
     </inertial>
   </link>
+  <joint name="camera_joint" type="fixed">
+    <origin xyz="0.040 -0.011 0.130" rpy="0 0.174 0"/>
+    <parent link="base_link"/>
+    <child link="camera_link"/>
+  </joint>
+  <link name="camera_link">
+    <collision>
+      <origin xyz="0.005 0.011 0.013" rpy="0 0 0"/>
+      <geometry>
+        <box size="0.015 0.030 0.027"/>
+      </geometry>
+    </collision>
+  </link>
+  <joint name="camera_rgb_joint" type="fixed">
+    <origin xyz="0.003 0.011 0.009" rpy="0 0 0"/>
+    <parent link="camera_link"/>
+    <child link="camera_rgb_frame"/>
+  </joint>
+  <link name="camera_rgb_frame"/>
+  <joint name="camera_rgb_optical_joint" type="fixed">
+    <origin xyz="0 0 0" rpy="-1.57 0 -1.57"/>
+    <parent link="camera_rgb_frame"/>
+    <child link="camera_rgb_optical_frame"/>
+  </joint>
+  <link name="camera_rgb_optical_frame"/>
 </robot>

Commit message: modified camera angle,camera_visual true

File: turtlebot3_description/urdf/turtlebot3_burger.gazebo.xacro (robot description, xacro)
@@ -2,5 +2,5 @@
 <robot name="turtlebot3_burger_sim" xmlns:xacro="http://ros.org/wiki/xacro">
   <xacro:arg name="laser_visual" default="false"/>
-  <xacro:arg name="camera_visual" default="false"/>
+  <xacro:arg name="camera_visual" default="true"/>
   <xacro:arg name="imu_visual"   default="false"/>
   <gazebo reference="base_link">

File: turtlebot3_description/urdf/turtlebot3_burger.urdf.xacro (robot description, xacro)
@@ -168,5 +168,5 @@
   </link>
   <joint name="camera_joint" type="fixed">
-    <origin xyz="0.040 -0.011 0.130" rpy="0 0.174 0"/>
+    <origin xyz="0.040 -0.011 0.130" rpy="0 1.047 0"/>
     <parent link="base_link"/>
     <child link="camera_link"/>
